Commit message: change turtlebot

File: model/turtlebot.urdf (robot description, URDF)
Before this commit: robot turtlebot, 33 links, 32 joints
Links:
- removed link camera_depth_frame
- removed link camera_depth_optical_frame
- removed link camera_rgb_frame
- removed link camera_rgb_optical_frame
- removed link eyes
- removed link plate_top_link
- removed link pole_kinect_0_link
- removed link pole_kinect_1_link
- added link pole_top_4_link, mass 0.001; collision cylinder length=0.2032 radius=.006; visual mesh filename=turtlebot/turtlebot_description/meshes/stacks/hexagons/pole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
- added link pole_top_5_link, mass 0.001; collision cylinder length=0.2032 radius=.006; visual mesh filename=turtlebot/turtlebot_description/meshes/stacks/hexagons/pole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
- added link pole_top_6_link, mass 0.001; collision cylinder length=0.2032 radius=.006; visual mesh filename=turtlebot/turtlebot_description/meshes/stacks/hexagons/pole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
- added link pole_top_7_link, mass 0.001; collision cylinder length=0.2032 radius=.006; visual mesh filename=turtlebot/turtlebot_description/meshes/stacks/hexagons/pole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
Joints:
- removed joint camera_depth_joint
- removed joint camera_depth_optical_joint
- removed joint camera_joint
- removed joint camera_rgb_joint
- removed joint camera_rgb_optical_joint
- removed joint plate_top_joint
- removed joint pole_kinect_0_joint
- removed joint pole_kinect_1_joint
- added joint pole_top_4_joint: type fixed, parent base_link, child pole_top_4_link, origin xyz=0.1024 0.098 0.2372 rpy=0 0 0
- added joint pole_top_5_joint: type fixed, parent base_link, child pole_top_5_link, origin xyz=0.1024 -0.098 0.2372 rpy=0 0 0
- added joint pole_top_6_joint: type fixed, parent base_link, child pole_top_6_link, origin xyz=-0.1024 0.098 0.2372 rpy=0 0 0
- added joint pole_top_7_joint: type fixed, parent base_link, child pole_top_7_link, origin xyz=-0.1024 -0.098 0.2372 rpy=0 0 0
- joint pole_top_0_joint: origin xyz=0.0381 0.1505 0.292 rpy=0 0 0 -> xyz=0.0381 0.1505 0.2372 rpy=0 0 0
- joint pole_top_1_joint: origin xyz=0.0381 -0.1505 0.292 rpy=0 0 0 -> xyz=0.0381 -0.1505 0.2372 rpy=0 0 0
- joint pole_top_2_joint: origin xyz=-0.0381 0.1505 0.292 rpy=0 0 0 -> xyz=-0.0381 0.1505 0.2372 rpy=0 0 0
- joint pole_top_3_joint: origin xyz=-0.0381 -0.1505 0.292 rpy=0 0 0 -> xyz=-0.0381 -0.1505 0.2372 rpy=0 0 0
